File: lora_board.kicad_pcb (KiCad board)
At the start: 2 copper layers, 22 x 60 mm, 12 parts, among them J1 Conn_01x03, J13 panel mount SMA, J2 I2C, J3 UART, U1 E22-900M22S, U2 ESP32-C3_SUPERMINI_SMD

Commit message: pre del
Parts:
- added C2: 10uF, Capacitor_SMD:C_1206_3216Metric_Pad1.33x1.80mm_HandSolder, B.Cu at (232.5, 127.0)
- added C3: 10uF, Capacitor_SMD:C_1206_3216Metric_Pad1.33x1.80mm_HandSolder, B.Cu at (270.5, 142.2)
- added C4: 10uF, Capacitor_SMD:C_1206_3216Metric_Pad1.33x1.80mm_HandSolder, F.Cu at (17.0, 142.0)
- added C4: 10uF, Capacitor_SMD:C_1206_3216Metric_Pad1.33x1.80mm_HandSolder, F.Cu at (183.8, 112.0)
- added C5: 10uF, Capacitor_SMD:C_1206_3216Metric_Pad1.33x1.80mm_HandSolder, F.Cu at (17.0, 144.5)
- added C5: 10uF, Capacitor_SMD:C_1206_3216Metric_Pad1.33x1.80mm_HandSolder, F.Cu at (183.8, 114.5)
- added C6: 10uF, Capacitor_SMD:C_1206_3216Metric_Pad1.33x1.80mm_HandSolder, F.Cu at (54.0, 81.5)
- added C6: 10uF, Capacitor_SMD:C_1206_3216Metric_Pad1.33x1.80mm_HandSolder, F.Cu at (183.8, 125.5)
- added C7: 10uF, Capacitor_SMD:C_1206_3216Metric_Pad1.33x1.80mm_HandSolder, F.Cu at (51.0, 143.0)
- added C7: 10uF, Capacitor_SMD:C_1206_3216Metric_Pad1.33x1.80mm_HandSolder, F.Cu at (183.8, 123.0)
- added C8: 10uF, Capacitor_SMD:C_1206_3216Metric_Pad1.33x1.80mm_HandSolder, F.Cu at (17.0, 147.0)
- added C8: 10uF, Capacitor_SMD:C_1206_3216Metric_Pad1.33x1.80mm_HandSolder, F.Cu at (183.8, 117.0)
- added D1: LED, LED_THT:LED_D3.0mm, B.Cu at (21.5, 87.8)
- added H3: MountingHole, MountingHole:MountingHole_2.2mm_M2_Pad_Via, F.Cu at (170.0, 114.0)
- added J10: BOOT, Connector_PinHeader_2.54mm:PinHeader_1x02_P2.54mm_Vertical, B.Cu at (27.0, 156.0)
- added J10: BOOT, Connector_PinHeader_2.54mm:PinHeader_1x02_P2.54mm_Vertical, B.Cu at (159.0, 128.0)
- added J11: RST, Connector_PinHeader_2.54mm:PinHeader_1x02_P2.54mm_Vertical, B.Cu at (170.3, 138.2)
- added J11: RST, Connector_PinHeader_2.54mm:PinHeader_1x02_P2.54mm_Vertical, B.Cu at (21.0, 156.0)
- added J4: Conn_Coaxial, Connector_Coaxial:SMA_Amphenol_132289_EdgeMount, F.Cu at (28.7, 82.5)
- added J4: Conn_Coaxial, Connector_Coaxial:SMA_Amphenol_132289_EdgeMount, F.Cu at (158.7, 82.5)
- added J4: Conn_Coaxial, Connector_Coaxial:SMA_Amphenol_132289_EdgeMount, B.Cu at (239.8, 117.0)
- added J5: USB_C_Receptacle_USB2.0_16P, Library:USB_C_Receptacle_GCT_USB4105-xx-A_16P_TopMnt_Horizontal, F.Cu at (184.2, 137.4)
- added J5: USB_C_Receptacle_USB2.0_16P, Library:USB_C_Receptacle_GCT_USB4105-xx-A_16P_TopMnt_Horizontal, B.Cu at (23.0, 95.5)
- added J6: Conn_01x10, Connector_PinHeader_2.54mm:PinHeader_1x10_P2.54mm_Vertical, B.Cu at (151.8, 138.2)
- added J7: Conn_01x10, Connector_PinHeader_2.54mm:PinHeader_1x10_P2.54mm_Vertical, B.Cu at (177.2, 138.2)
- added J8: Conn_01x04, Library:SSD1306-0.91-OLED-4pin-128x32, F.Cu at (151.5, 109.8)
- added J8: Conn_01x04, Library:SSD1306-0.91-OLED-4pin-128x32, B.Cu at (94.0, 99.5)
- added J9: Conn_01x03, Connector_PinHeader_2.54mm:PinHeader_1x03_P2.54mm_Vertical, F.Cu at (188.0, 130.0)
- added J9: Conn_01x03, Connector_Harwin:Harwin_M20-89003xx_1x03_P2.54mm_Horizontal, B.Cu at (49.5, 105.5)
- added JP1: SolderJumper_2_Open, Jumper:SolderJumper-2_P1.3mm_Open_RoundedPad1.0x1.5mm, F.Cu at (268.0, 137.8)
- added R2: 100k, Resistor_SMD:R_0603_1608Metric_Pad0.98x0.95mm_HandSolder, F.Cu at (182.2, 120.8)
- added R2: 100k, Resistor_SMD:R_0603_1608Metric_Pad0.98x0.95mm_HandSolder, F.Cu at (44.0, 147.0)
- added REF**: SOT-223, Package_TO_SOT_SMD:SOT-223, B.Cu at (233.5, 134.5)
- added REF**: PinHeader_1x04_P2.54mm_Vertical, Connector_PinHeader_2.54mm:PinHeader_1x04_P2.54mm_Vertical, B.Cu at (30.5, 99.3)
- added REF**: E22-900MM22S, Library:E22-900MM22S, B.Cu at (242.2, 126.5)
- added SW1: SW_Push, Button_Switch_SMD:SW_SPST_CK_RS282G05A3, B.Cu at (25.8, 104.0)
- added U2: ESP32-C3_SUPERMINI_SMD, Library:MODULE_ESP32-C3_SUPERMINI, F.Cu at (240.8, 129.0)
- added U3: SRV05-4, Package_TO_SOT_SMD:SOT-23-6_Handsoldering, F.Cu at (182.2, 129.2)
- added U3: SRV05-4, Package_TO_SOT_SMD:SOT-23-6_Handsoldering, F.Cu at (36.0, 147.0)
- added U4: E22P-868M30S, Library:E22P-868M30S, F.Cu at (40.0, 96.8)
- added U4: E22P-868M30S, Library:E22P-868M30S, F.Cu at (170.0, 96.8)
- added U5: ESP32-S3-WROOM-1, Library:ESP32-S3-WROOM-1, F.Cu at (164.5, 133.8)
- added U5: ESP32-S3-WROOM-1, Library:ESP32-S3-WROOM-1, B.Cu at (49.0, 86.2)
- J2: moved to F.Cu
- moved J2 118.1 mm to (46.9, 28.7), turned to 0 degrees
Routing:
- net +3V3: track 55.4 -> 160.4 mm, vias 4 -> 7
- net +5V: track 38.2 -> 132.1 mm
- net /USB_D+: track 0.00 -> 81.0 mm
- net /USB_D-: track 0.00 -> 81.0 mm
- net /CS: track 46.7 -> 117.3 mm, vias 2 -> 5
- net /IRQ: track 38.8 -> 107.4 mm, vias 2 -> 5
- net /BUSY: track 28.0 -> 96.1 mm, vias 2 -> 5
- net /RST: track 33.5 -> 98.5 mm, vias 2 -> 5
- net /MISO: track 46.3 -> 109.2 mm, vias 2 -> 5
- net /MOSI: track 45.6 -> 108.1 mm, vias 2 -> 5
- net /SCK: track 44.0 -> 106.4 mm, vias 2 -> 5
- net /SDA: track 8.79 -> 70.3 mm, vias 0 -> 2
- net /SCL: track 12.4 -> 72.1 mm, vias 0 -> 2
- net /EN: track 0.00 -> 24.4 mm, vias 0 -> 2
- net /GPIO17: track 0.00 -> 16.0 mm, vias 0 -> 1
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- added copper zone on B.Cu, net /LORA_EN
Other:
- board size 22 x 60 mm -> 230 x 60 mm
- board text added: "${REFERENCE}"
- board text added: "1"
- board text added: "15"
- board text added: "16"
- board text added: "17"
- board text added: "2"
- board text added: "3"
- board text added: "39"
- board text added: "3V3"
- board text added: "4"
- board text added: "40"
- board text added: "41"
- board text added: "42"
- board text added: "5"
- board text added: "5V"
- board text added: "6"
- board text added: "7"
- board text added: "ESP32-S3-WROOM-1 E22P-868M30S LORA base v1"
- board text added: "GND"
- board text added: "RX"
- board text added: "TX"

Commit message: pre del esp32-s3-supermini
Parts:
- removed C1, C4 (x2), C5 (x2), C6 (x2), C7 (x2), C8 (x2): 10uF, Capacitor_SMD:C_1206_3216Metric_Pad1.33x1.80mm_HandSolder
- removed the C2 at (91.0, 110.2)
- removed the C3 at (103.5, 112.8)
- removed D1: LED, LED_THT:LED_D3.0mm
- removed H3: MountingHole, MountingHole:MountingHole_2.2mm_M2_Pad_Via
- removed J1, J9: Conn_01x03, Connector_PinHeader_2.54mm:PinHeader_1x03_P2.54mm_Vertical
- removed J10 (x2): BOOT, Connector_PinHeader_2.54mm:PinHeader_1x02_P2.54mm_Vertical
- removed J11 (x2): RST, Connector_PinHeader_2.54mm:PinHeader_1x02_P2.54mm_Vertical
- removed J13: panel mount SMA, Connector_Coaxial:SMA_Amphenol_901-143_Horizontal
- removed J2: I2C, Connector_PinHeader_2.54mm:PinHeader_1x04_P2.54mm_Vertical
- removed J4 (x3): Conn_Coaxial, Connector_Coaxial:SMA_Amphenol_132289_EdgeMount
- removed J5 (x2): USB_C_Receptacle_USB2.0_16P, Library:USB_C_Receptacle_GCT_USB4105-xx-A_16P_TopMnt_Horizontal
- removed J6, J7: Conn_01x10, Connector_PinHeader_2.54mm:PinHeader_1x10_P2.54mm_Vertical
- removed J8 (x2): Conn_01x04, Library:SSD1306-0.91-OLED-4pin-128x32
- removed J9: Conn_01x03, Connector_Harwin:Harwin_M20-89003xx_1x03_P2.54mm_Horizontal
- removed JP1 (x2): SolderJumper_2_Open, Jumper:SolderJumper-2_P1.3mm_Open_RoundedPad1.0x1.5mm
- removed the R2 at (182.2, 120.8)
- removed the R2 at (44.0, 147.0)
- removed the REF** at (233.5, 134.5)
- removed the REF** at (30.5, 99.3)
- removed the REF** at (242.2, 126.5)
- removed U2 (x2): ESP32-C3_SUPERMINI_SMD, Library:MODULE_ESP32-C3_SUPERMINI
- removed the U3 at (182.2, 129.2)
- removed the U3 at (36.0, 147.0)
- removed U4 (x2): E22P-868M30S, Library:E22P-868M30S
- removed U5 (x2): ESP32-S3-WROOM-1, Library:ESP32-S3-WROOM-1
- added AE1: Antenna_Shield, Connector_Coaxial:SMA_Amphenol_132289_EdgeMount, B.Cu at (141.5, 93.0)
- added AE1: Antenna_Shield, Connector_Coaxial:SMA_Amphenol_132289_EdgeMount, B.Cu at (105.0, 77.5)
- added R1: R, Resistor_SMD:R_0603_1608Metric_Pad0.98x0.95mm_HandSolder, F.Cu at (145.2, 98.8)
- added R2: R, Resistor_SMD:R_0603_1608Metric_Pad0.98x0.95mm_HandSolder, F.Cu at (145.2, 101.3)
- added REF**: USB_C_Receptacle_GCT_USB4105-xx-A_16P_TopMnt_Horizontal, Connector_USB:USB_C_Receptacle_GCT_USB4105-xx-A_16P_TopMnt_Horizontal, B.Cu at (104.8, 113.0)
- added REF**: SW_SPDT_PCM12, Button_Switch_SMD:SW_SPDT_PCM12, B.Cu at (96.8, 79.2)
- added REF**: E73-2G4M08S1C, Library:E73-2G4M08S1C, B.Cu at (104.2, 101.2)
- added U3: E22-900MM22S, Library:E22-900MM22S, B.Cu at (144.0, 102.5)
- added U3: E22-900MM22S, Library:E22-900MM22S, B.Cu at (108.0, 87.0)
- C2: moved to F.Cu
- C3: value 10uF -> 100nF; footprint Capacitor_SMD:C_1206_3216Metric_Pad1.33x1.80mm_HandSolder -> Capacitor_SMD:C_0603_1608Metric_Pad1.08x0.95mm_HandSolder; moved to F.Cu
- SW1: value SW_Push -> SW_Slide_DPDT; footprint Button_Switch_SMD:SW_SPST_CK_RS282G05A3 -> Button_Switch_THT:SW_CK_JS202011AQN_DPDT_Angled; moved to F.Cu
- U1: value E22-900M22S -> ESP32-S3_SUPERMINI_SMD; footprint Library:E22-900M22S -> Library:MODULE_ESP32-S3_SUPERMINI
- moved C3 135.0 mm to (145.5, 91.2), turned to 0 degrees
- moved H1 124.5 mm to (216.0, 99.5)
- moved SW1 123.8 mm to (148.5, 88.0), turned to 90 degrees
- moved H2 110.7 mm to (216.0, 105.4)
- moved C2 93.6 mm to (145.0, 93.8), turned to 0 degrees
- moved J3 50.6 mm to (149.3, 114.5), turned to 90 degrees
- moved U1 44.5 mm to (141.5, 114.5), turned to 90 degrees
Connections:
- C2 pad 1: +3.3V -> /E22_VCC
- C3 pad 1: +3V3 -> /E22_VCC
- SW1 pad 1: GND -> /ESP_RST
- SW1 pad 2: unconnected-(SW1-Pad2) -> GND
- U1 pad 1: GND -> unconnected-(U1-GPIO10-Pad1)
- U1 pad 10: GND -> /SCK
- U1 pad 11: GND -> /CS
- U1 pad 12: GND -> /MOSI
- U1 pad 13: /IRQ -> /MISO
- U1 pad 15: /RST -> unconnected-(U1-B--Pad15)
- U1 pad 16: /MISO -> /BAT+
- U1 pad 2: GND -> unconnected-(U1-GPIO11-Pad2)
- U1 pad 21: unconnected-(U1-ANT-Pad21) -> (no net)
- U1 pad 3: GND -> unconnected-(U1-GPIO12-Pad3)
- U1 pad 4: GND -> unconnected-(U1-GPIO13-Pad4)
- U1 pad 5: GND -> /TX
- U1 pad 6: /RXEN -> /RX
- U1 pad 7: /TXEN -> /E22_RST
- U1 pad 8: /TXEN -> /IRQ
- U1 pad 9: +3.3V -> unconnected-(U1-GPIO3-Pad9)
Routing:
- net +3V3: track 160.4 -> 0.00 mm, vias 7 -> 0
- net +5V: track 132.1 -> 0.00 mm, vias 4 -> 0
- net /CS: track 117.3 -> 0.00 mm, vias 5 -> 0
- net /MISO: track 109.2 -> 0.00 mm, vias 5 -> 0
- net /MOSI: track 108.1 -> 0.00 mm, vias 5 -> 0
- net /IRQ: track 107.4 -> 0.00 mm, vias 5 -> 0
- net /SCK: track 106.4 -> 0.00 mm, vias 5 -> 0
- net /RST: track 98.5 -> 0.00 mm, vias 5 -> 0
- net /BUSY: track 96.1 -> 0.00 mm, vias 5 -> 0
- net /USB_D+: track 81.0 -> 0.00 mm
- net /USB_D-: track 81.0 -> 0.00 mm
- net /SCL: track 72.1 -> 0.00 mm, vias 2 -> 0
- net /SDA: track 70.3 -> 0.00 mm, vias 2 -> 0
- net /RXEN: track 29.4 -> 0.00 mm, vias 2 -> 0
- net +3.3V: track 25.6 -> 0.00 mm
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- added copper zone on F.Cu, net /ANT
- removed copper zone on B.Cu, net /LORA_EN
Other:
- board size 230 x 60 mm -> 58 x 50 mm
- board text removed: "1"
- board text removed: "15"
- board text removed: "16"
- board text removed: "17"
- board text removed: "2"
- board text removed: "3"
- board text removed: "39"
- board text removed: "3V3"
- board text removed: "4"
- board text removed: "40"
- board text removed: "41"
- board text removed: "42"
- board text removed: "5"
- board text removed: "5V"
- board text removed: "6"
- board text removed: "7"
- board text removed: "ESP32-C3 E22-900M22S LORA v1"
- board text removed: "ESP32-S3-WROOM-1 E22P-868M30S LORA base v1"
- board text removed: "GND"
- board text removed: "RX"
- board text removed: "TX"

Commit message: small ordered v1
Parts:
- removed the AE1 at (141.5, 93.0)
- removed H1, H2: MountingHole, MountingHole:MountingHole_2.2mm_M2_Pad_Via
- removed REF**: USB_C_Receptacle_GCT_USB4105-xx-A_16P_TopMnt_Horizontal, Connector_USB:USB_C_Receptacle_GCT_USB4105-xx-A_16P_TopMnt_Horizontal
- removed REF**: SW_SPDT_PCM12, Button_Switch_SMD:SW_SPDT_PCM12
- removed REF**: E73-2G4M08S1C, Library:E73-2G4M08S1C
- removed the U3 at (144.0, 102.5)
- added C1: 10uF, Capacitor_SMD:C_0603_1608Metric_Pad1.08x0.95mm_HandSolder, F.Cu at (109.0, 86.2)
- added C4: 10uF, Capacitor_SMD:C_0603_1608Metric_Pad1.08x0.95mm_HandSolder, F.Cu at (113.0, 88.8)
- added C5: 10uF, Capacitor_SMD:C_0603_1608Metric_Pad1.08x0.95mm_HandSolder, F.Cu at (113.0, 111.8)
- added C6: 10uF, Capacitor_SMD:C_0603_1608Metric_Pad1.08x0.95mm_HandSolder, F.Cu at (109.5, 111.8)
- added D1: LED, LED_SMD:LED_0603_1608Metric_Pad1.05x0.95mm_HandSolder, F.Cu at (113.0, 119.0)
- added D2: LED, LED_SMD:LED_0603_1608Metric_Pad1.05x0.95mm_HandSolder, F.Cu at (97.0, 119.0)
- added D3: LED, LED_SMD:LED_0603_1608Metric_Pad1.05x0.95mm_HandSolder, F.Cu at (97.2, 76.2)
- added J1: USB_C_Receptacle_USB2.0_16P, Connector_USB:USB_C_Receptacle_GCT_USB4105-xx-A_16P_TopMnt_Horizontal, F.Cu at (104.5, 117.5)
- added J2: Conn_01x02_Shielded, Connector_JST:JST_SH_SM02B-SRSS-TB_1x02-1MP_P1.00mm_Horizontal, F.Cu at (111.5, 92.2)
- added J4: Conn_01x02, Library:1x02 smd 2.54, B.Cu at (105.0, 117.5)
- added L1: 10uH, Inductor_SMD:L_0603_1608Metric_Pad1.05x0.95mm_HandSolder, F.Cu at (97.0, 110.0)
- added R10: 5.1k, Resistor_SMD:R_0603_1608Metric_Pad0.98x0.95mm_HandSolder, F.Cu at (97.0, 111.5)
- added R3: 1k, Resistor_SMD:R_0603_1608Metric_Pad0.98x0.95mm_HandSolder, F.Cu at (97.0, 117.5)
- added R4: 5.1k, Resistor_SMD:R_0603_1608Metric_Pad0.98x0.95mm_HandSolder, F.Cu at (110.5, 118.0)
- added R5: 5.1k, Resistor_SMD:R_0603_1608Metric_Pad0.98x0.95mm_HandSolder, F.Cu at (109.0, 82.8)
- added R6: 1k, Resistor_SMD:R_0603_1608Metric_Pad0.98x0.95mm_HandSolder, F.Cu at (113.0, 117.2)
- added R7: 1k, Resistor_SMD:R_0603_1608Metric_Pad0.98x0.95mm_HandSolder, F.Cu at (97.2, 77.8)
- added R8: 5.1k, Resistor_SMD:R_0603_1608Metric_Pad0.98x0.95mm_HandSolder, F.Cu at (106.0, 111.8)
- added R9: 5.1k, Resistor_SMD:R_0603_1608Metric_Pad0.98x0.95mm_HandSolder, F.Cu at (101.0, 111.8)
- added SW2: SW_SPDT, Button_Switch_SMD:SW_SPDT_PCM12, F.Cu at (112.8, 79.8)
- added U2: AP2112K-3.3, Package_TO_SOT_SMD:SOT-23-5_HandSoldering, F.Cu at (112.0, 86.0)
- added U4: MCP73831-2-OT, Package_TO_SOT_SMD:SOT-23-5_HandSoldering, F.Cu at (112.2, 114.5)
- AE1: moved to F.Cu
- C2: value 10uF -> 100nF; footprint Capacitor_SMD:C_1206_3216Metric_Pad1.33x1.80mm_HandSolder -> Capacitor_SMD:C_0603_1608Metric_Pad1.08x0.95mm_HandSolder
- J3: value UART -> Conn_01x05; footprint Connector_PinHeader_2.54mm:PinHeader_1x04_P2.54mm_Vertical -> Connector_PinHeader_2.54mm:PinHeader_1x05_P2.54mm_Vertical
- R1, R2: value R -> 1M
- SW1: value SW_Slide_DPDT -> SW_Push; footprint Button_Switch_THT:SW_CK_JS202011AQN_DPDT_Angled -> Button_Switch_SMD:SW_SPST_B3U-1000P
- U1: value ESP32-S3_SUPERMINI_SMD -> E73-2G4M08S1C; footprint Library:MODULE_ESP32-S3_SUPERMINI -> Library:E73-2G4M08S1C
- U3: footprint Library:E22-900MM22S -> Library:E22-900MM22S_handsolder; moved to F.Cu
- moved SW1 57.9 mm to (97.0, 114.5)
- moved R2 48.7 mm to (97.2, 93.2), turned to 180 degrees
- moved R1 48.2 mm to (97.2, 94.8)
- moved C2 44.0 mm to (101.0, 93.8)
- moved J3 40.9 mm to (110.1, 103.0)
- moved U1 37.3 mm to (106.0, 103.0), turned to -90 degrees
- moved C3 36.1 mm to (109.5, 88.8)
- moved U3 6.54 mm to (101.5, 86.2), turned to 180 degrees
Connections:
- AE1 pad 1: (no net) -> /ANT
- AE1 pad 2: (no net) -> GND
- C2 pad 1: /E22_VCC -> /BAT_SENSE
- C3 pad 1: /E22_VCC -> +3.3V
- J3 pad 2: /RX -> /SWDCLK
- J3 pad 3: /TX -> /SWDIO
- J3 pad 4: +3.3V -> /NRF_RESET
- R1 pad 1: /BAT+ -> VCC
- SW1 pad 1: /ESP_RST -> GND
- SW1 pad 2: GND -> /NRF_RESET
- U1 pad 1: unconnected-(U1-GPIO10-Pad1) -> /E22_RST
- U1 pad 11: /CS -> unconnected-(U1B-P0.00/XL1-Pad11)
- U1 pad 13: /MISO -> unconnected-(U1B-P0.01/XL2-Pad13)
- U1 pad 15: unconnected-(U1-B--Pad15) -> /LED
- U1 pad 21: (no net) -> GND
- U1 pad 25: (no net) -> Net-(U1A-DCCH)
- U1 pad 26: (no net) -> /NRF_RESET
- U1 pad 27: (no net) -> +5V
- U1 pad 3: unconnected-(U1-GPIO12-Pad3) -> /IRQ
- U1 pad 33: (no net) -> unconnected-(U1B-P0.13-Pad33)
- U1 pad 35: (no net) -> unconnected-(U1B-P0.24-Pad35)
- U1 pad 37: (no net) -> /SWDIO
- U1 pad 39: (no net) -> /SWDCLK
- U1 pad 4: unconnected-(U1-GPIO13-Pad4) -> /BAT_SENSE
- U1 pad 41: (no net) -> unconnected-(U1B-P0.09/NFC1-Pad41)
- U1 pad 5: /TX -> GND
- U1 pad 6: /RX -> /BUSY
- U1 pad 7: /E22_RST -> /MISO
- U1 pad 8: /IRQ -> /MOSI
- U1 pad 9: unconnected-(U1-GPIO3-Pad9) -> /CS
- U3 pad 1: (no net) -> +3.3V
- U3 pad 10: (no net) -> /RXEN
- U3 pad 11: (no net) -> /BUSY
- U3 pad 12: (no net) -> /MISO
- U3 pad 13: (no net) -> /MOSI
- U3 pad 14: (no net) -> /CS
- U3 pad 15: (no net) -> /SCK
- U3 pad 16: (no net) -> GND
- U3 pad 17: (no net) -> unconnected-(U3-NC-Pad17)
- U3 pad 18: (no net) -> unconnected-(U3-DIO3-Pad18)
- U3 pad 19: (no net) -> /TXEN
- U3 pad 2: (no net) -> GND
- U3 pad 20: (no net) -> /IRQ
- U3 pad 3: (no net) -> /E22_RST
- U3 pad 4: (no net) -> unconnected-(U3-NC-Pad4)
- U3 pad 5: (no net) -> unconnected-(U3-NC-Pad5)
- U3 pad 6: (no net) -> /ANT
- U3 pad 7: (no net) -> GND
- U3 pad 8: (no net) -> unconnected-(U3-NC-Pad8)
- U3 pad 9: (no net) -> /TXEN
Routing:
- net VCC: track 0.00 -> 63.5 mm, vias 0 -> 4
- net +BATT: track 0.00 -> 42.2 mm, vias 0 -> 3
- net /LED: track 0.00 -> 26.4 mm, vias 0 -> 2
- net /RXEN: track 0.00 -> 24.9 mm, vias 0 -> 2
- net /BUSY: track 0.00 -> 20.7 mm, vias 0 -> 2
- net /MISO: track 0.00 -> 18.9 mm, vias 0 -> 2
- net +5V: track 0.00 -> 18.5 mm, vias 0 -> 1
- net /MOSI: track 0.00 -> 17.2 mm, vias 0 -> 2
- net /E22_RST: track 0.00 -> 15.6 mm
- net /CS: track 0.00 -> 15.4 mm, vias 0 -> 2
- net /SCK: track 0.00 -> 14.2 mm, vias 0 -> 2
- net VDD: track 0.00 -> 13.6 mm
- net /BAT_SENSE: track 0.00 -> 13.4 mm
- net /NRF_RESET: track 0.00 -> 12.8 mm
- net /TXEN: track 0.00 -> 11.3 mm
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Other:
- board size 58 x 50 mm -> 20 x 45 mm
- board text added: "+"
- board text added: "-"
- board text added: "3V3"
- board text added: "GND"
- board text added: "LORA Small v2"
- board text added: "RST"
- board text added: "SWC"
- board text added: "SWI"
- board text removed: "${REFERENCE}"

Commit message: v2 rc1
Parts:
- removed D3: LED, LED_SMD:LED_0603_1608Metric_Pad1.05x0.95mm_HandSolder
- removed the R7 at (97.2, 77.8)
- added BZ1: Buzzer, Library:MLT-5020, F.Cu at (98.5, 87.0)
- added C7: 10uF, Capacitor_SMD:C_0603_1608Metric_Pad1.08x0.95mm_HandSolder, F.Cu at (96.0, 91.2)
- added Q1: AO3400A, Package_TO_SOT_SMD:SOT-23_Handsoldering, F.Cu at (99.2, 91.2)
- C1: renamed from C3; footprint Capacitor_SMD:C_0603_1608Metric_Pad1.08x0.95mm_HandSolder -> Capacitor_SMD:C_0402_1005Metric_Pad0.74x0.62mm_HandSolder
- C2: footprint Capacitor_SMD:C_0603_1608Metric_Pad1.08x0.95mm_HandSolder -> Capacitor_SMD:C_0402_1005Metric_Pad0.74x0.62mm_HandSolder
- R5: value 5.1k -> 10k
- R6: renamed from R10; value 5.1k -> 10k
- moved R1 19.7 mm to (105.8, 77.0), turned to -90 degrees
- moved R5 17.7 mm to (97.0, 95.8), turned to 180 degrees
- moved C4 16.8 mm to (97.0, 94.0)
- moved R2 15.8 mm to (105.0, 79.5)
- moved J2 14.9 mm to (100.8, 82.0), turned to -90 degrees
- moved SW2 12.8 mm to (100.2, 77.0), turned to 180 degrees
- moved U2 11.9 mm to (102.8, 93.5), turned to 0 degrees
- moved C3 7.89 mm to (110.5, 94.0), turned to 180 degrees
- moved U3 7.00 mm to (108.5, 86.5)
- moved C2 5.76 mm to (106.8, 94.0), turned to 180 degrees
- moved AE1 5.50 mm to (110.5, 77.5)
- moved C1 4.78 mm to (113.0, 92.0), turned to 180 degrees
- turned D1 to 180 degrees
- turned D2 to 180 degrees
- turned R4 to 180 degrees
- renumbered C1 to C3, R6 to R4, R4 to R7
Connections:
- D1 pad 1: GND -> Net-(D1-K)
- D1 pad 2: Net-(D1-A) -> +5V
- J2 pad MP: (no net) -> GND
- R3 pad 1: VCC -> /LED
- R4 pad 1: Net-(U4-STAT) -> Net-(D1-K)
- R4 pad 2: Net-(D1-A) -> /STAT
- U1 pad 2: unconnected-(U1C-P1.10-Pad2) -> /BUZZER
- U1 pad 33: unconnected-(U1B-P0.13-Pad33) -> /REG_EN
- U4 pad 1: Net-(U4-STAT) -> /STAT
Routing:
- net +3.3V: track 5.77 -> 28.9 mm
- net /BUZZER: track 0.00 -> 21.9 mm, vias 0 -> 2
- net VCC: track 63.5 -> 44.1 mm, vias 4 -> 3
- net /REG_EN: track 4.71 -> 23.2 mm
- net /RXEN: track 24.9 -> 33.5 mm
- net +5V: track 18.5 -> 26.8 mm
- net /BAT_SENSE: track 13.4 -> 21.1 mm, vias 0 -> 2
- net /LED: track 26.4 -> 19.1 mm
- net +BATT: track 42.2 -> 47.3 mm, vias 3 -> 4
- net /SCK: track 14.2 -> 10.8 mm
- net Net-(U4-STAT): track 2.55 -> 0.00 mm
- net /BUSY: track 20.7 -> 18.2 mm
- net /STAT: track 0.00 -> 2.52 mm
- net Net-(BZ1--): track 0.00 -> 2.52 mm
- net /IRQ: track 8.35 -> 10.8 mm, vias 0 -> 2
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Other:
- outline, holes or cut-outs redrawn

Commit message: v2 rc2
Parts:
- J4: value Conn_01x02 -> Qi Charger; footprint Library:1x02 smd 2.54 -> Library:QiCharger
- R3: renamed from R5; value 10k -> 1M
- R4: value 1k -> 330
- R5: renamed from R3; value 1k -> 330
- R6: value 10k -> 5.1k
- U3: footprint Library:E22-900MM22S_handsolder -> Library:E22-900MM22S
- moved J4 37.5 mm to (105.5, 80.0)
- moved C1 3.20 mm to (110.5, 94.0), turned to -90 degrees
- moved C3 1.25 mm to (109.2, 94.0), turned to -90 degrees
- moved U3 0.56 mm to (109.0, 86.2)
- moved AE1 0.50 mm to (111.0, 77.5)
- moved J3 0.50 mm to (110.6, 103.0)
- moved R2 0.50 mm to (105.5, 79.5)
- moved C6 0.25 mm to (109.5, 111.5)
- moved J1 0.25 mm to (104.2, 117.5)
- moved J2 0.25 mm to (101.0, 82.0)
- moved R1 0.25 mm to (106.0, 77.0)
- moved R8 0.25 mm to (106.0, 111.5)
- moved R9 0.25 mm to (101.0, 111.5)
- moved SW2 0.25 mm to (100.0, 77.0)
- moved U1 0.25 mm to (105.8, 103.0)
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Connections:
- R3 pad 1: /REG_EN -> GND
- R3 pad 2: VCC -> /REG_EN
- U3 pad 17: unconnected-(U3-NC-Pad17) -> GND
- U3 pad 4: unconnected-(U3-NC-Pad4) -> GND
- U3 pad 5: unconnected-(U3-NC-Pad5) -> GND
- U3 pad 8: unconnected-(U3-NC-Pad8) -> GND
Routing:
- net +5V: track 26.8 -> 68.3 mm
- net GND: track 2.72 -> 0.00 mm, vias 45 -> 46
- net +3.3V: track 28.9 -> 26.9 mm
- net VCC: track 44.1 -> 42.1 mm
- net +BATT: track 47.3 -> 49.2 mm
- net /BAT_SENSE: track 21.1 -> 22.9 mm
- net /BUZZER: track 21.9 -> 21.0 mm
- net Net-(D2-A): track 2.33 -> 1.52 mm
- net Net-(BZ1--): track 2.52 -> 3.26 mm
- net /SCK: track 10.8 -> 11.6 mm
- net VDD: track 13.6 -> 14.3 mm
- net /RXEN: track 33.5 -> 33.0 mm
Other:
- outline, holes or cut-outs redrawn
- board text added: ">"
- board text added: "LSBN v2"
- board text added: "SWCLK"
- board text added: "SWIO"
- board text added: "VREF"
- board text removed: "+"
- board text removed: "-"
- board text removed: "3V3"
- board text removed: "LORA Small v2"
- board text removed: "SWC"
- board text removed: "SWI"
