File: lora_board.kicad_sch (KiCad schematic)
At the start: 12 parts, among them J1 Conn_01x03, J13 panel mount SMA, J2 I2C, J3 UART, U1 E22-900M22S, U2 ESP32-C3_SUPERMINI_SMD

Commit message: pre del
Parts:
- added C4, C5, C6, C7, C8: 10uF, Capacitor_SMD:C_1206_3216Metric_Pad1.33x1.80mm_HandSolder, symbol Device:C
- added D1: LED, LED_THT:LED_D3.0mm, symbol Device:LED
- added H3: MountingHole, MountingHole:MountingHole_2.2mm_M2_Pad_Via, symbol Mechanical:MountingHole
- added J10: BOOT, Connector_PinHeader_2.54mm:PinHeader_1x02_P2.54mm_Vertical, symbol Connector_Generic:Conn_01x02
- added J11: RST, Connector_PinHeader_2.54mm:PinHeader_1x02_P2.54mm_Vertical, symbol Connector_Generic:Conn_01x02
- added J4: Conn_Coaxial, symbol Connector:Conn_Coaxial
- added J5: USB_C_Receptacle_USB2.0_16P, Library:USB_C_Receptacle_GCT_USB4105-xx-A_16P_TopMnt_Horizontal, symbol Connector:USB_C_Receptacle_USB2.0_16P
- added J6, J7: Conn_01x10, Connector_PinHeader_2.54mm:PinHeader_1x10_P2.54mm_Vertical, symbol Connector_Generic:Conn_01x10
- added J8: Conn_01x04, Library:SSD1306-0.91-OLED-4pin-128x32, symbol Connector_Generic:Conn_01x04
- added J9: Conn_01x03, Connector_PinHeader_2.54mm:PinHeader_1x03_P2.54mm_Vertical, symbol Connector_Generic:Conn_01x03
- added R1: R, symbol Device:R
- added R2: 100k, Resistor_SMD:R_0603_1608Metric_Pad0.98x0.95mm_HandSolder, symbol Device:R
- added SW1: SW_Push, Button_Switch_SMD:SW_SPST_CK_RS282G05A3, symbol Switch:SW_Push
- added U3: SRV05-4, Package_TO_SOT_SMD:SOT-23-6_Handsoldering, symbol Power_Protection:SRV05-4
- added U4: E22P-868M30S, E22-900M30S:XCVR_E22-900M30S, symbol New_Library:E22P-868M30S
- added U5: ESP32-S3-WROOM-1, Library:ESP32-S3-WROOM-1, symbol RF_Module:ESP32-S3-WROOM-1
Connections:
- net +3V3: now also C6.1, J7.2 (Pin_2), J8.2 (Pin_2), J9.2 (Pin_2), R2.1, U5.2 (3V3)
- net +5V: now also C4.1, C5.1, C7.1, C8.1, J5.A4 (VBUS), J5.A9 (VBUS), J5.B4 (VBUS), J5.B9 (VBUS), J7.3 (Pin_3), J9.3 (Pin_3), U3.5 (VP), U4.10 (VCC), U4.9 (VCC)
- net BUSY: now also U4.14 (BUSY), U5.23 (IO21)
- net CS: now also U4.19 (NSS), U5.18 (IO10)
- net GND: now also C4.2, C5.2, C6.2, C7.2, C8.2, D1.1 (K), J10.1 (Pin_1), J11.1 (Pin_1), J4.2 (Ext), J5.A1 (GND), J5.A12 (GND), J5.B1 (GND), J5.B12 (GND), J5.S1 (SHIELD), J6.1 (Pin_1), J7.1 (Pin_1), J8.1 (Pin_1), J9.1 (Pin_1), SW1.1, U3.2 (VN), U4.1 (GND), U4.11 (GND), U4.12 (GND), U4.2 (GND), U4.20 (GND), U4.22 (GND), U4.3 (GND), U4.4 (GND), U4.5 (GND), U5.1 (GND), U5.40 (GND), U5.41 (GND)
- net IRQ: now also U4.13 (DIO1), U5.22 (IO14)
- net MISO: now also U4.16 (MISO), U5.21 (IO13)
- net MOSI: now also U4.17 (MOSI), U5.19 (IO11)
- net RST: now also U4.15 (~{RST}), U5.17 (IO9)
- net SCK: now also U4.18 (SCK), U5.20 (IO12)
- net SCL: now also J8.3 (Pin_3), U5.12 (IO8)
- net SDA: now also J8.4 (Pin_4), U5.11 (IO18)
- new net: J4.1 (In), U4.21 (ANT)
- new net: D1.2 (A), R1.2
- new net BOOT0: J10.2 (Pin_2), U5.27 (IO0)
- new net BOOT1: U5.16 (IO46)
- new net BOOT2: U5.26 (IO45)
- new net EN: J11.2 (Pin_2), R2.2, U5.3 (EN)
- new net GPIO01: J6.2 (Pin_2), U5.39 (IO1)
- new net GPIO02: J6.3 (Pin_3), U5.38 (IO2)
- new net GPIO04: J7.4 (Pin_4), U5.4 (IO4)
- new net GPIO05: J7.5 (Pin_5), U5.5 (IO5)
- new net GPIO06: J7.6 (Pin_6), U5.6 (IO6)
- new net GPIO07: J7.7 (Pin_7), U5.7 (IO7)
- new net GPIO15: J7.8 (Pin_8), U5.8 (IO15)
- new net GPIO16: J7.9 (Pin_9), U5.9 (IO16)
- new net GPIO17: J7.10 (Pin_10), U5.10 (IO17)
- new net GPIO38: J6.10 (Pin_10), U5.31 (IO38)
- new net GPIO39: J6.9 (Pin_9), U5.32 (IO39)
- new net GPIO40: J6.8 (Pin_8), U5.33 (IO40)
- new net GPIO41: J6.7 (Pin_7), U5.34 (IO41)
- new net GPIO42: J6.6 (Pin_6), U5.35 (IO42)
- new net LORA_EN: U4.6 (EN), U5.15 (IO3)
- new net RXD: J6.5 (Pin_5), U5.36 (RXD0)
- new net TREN: U4.7 (T/R_EN), U4.8 (DIO2)
- new net TXD: J6.4 (Pin_4), U5.37 (TXD0)
- new net USB_D+: J5.A6 (D+), J5.B6 (D+), U3.1 (IO1), U3.3 (IO2), U5.14 (USB_D+)
- new net USB_D-: J5.A7 (D-), J5.B7 (D-), U3.4 (IO3), U3.6 (IO4), U5.13 (USB_D-)
- no-connect marks 4 -> 13
Other:
- note added: "1.8V"
- moved on the sheet: C1, C2, C3, H1, H2, J1, J13, J2, J3, JP1, U1, U2

Commit message: pre del esp32-s3-supermini
Parts:
- removed C1, C4, C5, C6, C7, C8: 10uF, Capacitor_SMD:C_1206_3216Metric_Pad1.33x1.80mm_HandSolder, symbol Device:C
- removed H3: MountingHole, MountingHole:MountingHole_2.2mm_M2_Pad_Via, symbol Mechanical:MountingHole
- removed J1, J9: Conn_01x03, Connector_PinHeader_2.54mm:PinHeader_1x03_P2.54mm_Vertical, symbol Connector_Generic:Conn_01x03
- removed J10: BOOT, Connector_PinHeader_2.54mm:PinHeader_1x02_P2.54mm_Vertical, symbol Connector_Generic:Conn_01x02
- removed J11: RST, Connector_PinHeader_2.54mm:PinHeader_1x02_P2.54mm_Vertical, symbol Connector_Generic:Conn_01x02
- removed J13: panel mount SMA, Connector_Coaxial:SMA_Amphenol_901-143_Horizontal, symbol Connector:Conn_Coaxial
- removed J2: I2C, Connector_PinHeader_2.54mm:PinHeader_1x04_P2.54mm_Vertical, symbol Connector_Generic:Conn_01x04
- removed J4: Conn_Coaxial, symbol Connector:Conn_Coaxial
- removed J5: USB_C_Receptacle_USB2.0_16P, Library:USB_C_Receptacle_GCT_USB4105-xx-A_16P_TopMnt_Horizontal, symbol Connector:USB_C_Receptacle_USB2.0_16P
- removed J6, J7: Conn_01x10, Connector_PinHeader_2.54mm:PinHeader_1x10_P2.54mm_Vertical, symbol Connector_Generic:Conn_01x10
- removed J8: Conn_01x04, Library:SSD1306-0.91-OLED-4pin-128x32, symbol Connector_Generic:Conn_01x04
- removed JP1: SolderJumper_2_Open, Jumper:SolderJumper-2_P1.3mm_Open_RoundedPad1.0x1.5mm, symbol Jumper:SolderJumper_2_Open
- removed SW1: SW_Push, Button_Switch_SMD:SW_SPST_CK_RS282G05A3, symbol Switch:SW_Push
- removed U1: E22-900M22S, Library:E22-900M22S, symbol New_Library:E22-900M22S
- removed U2: ESP32-C3_SUPERMINI_SMD, Library:MODULE_ESP32-C3_SUPERMINI, symbol ESP32-C3_SUPERMINI_SMD:ESP32-C3_SUPERMINI_SMD
- removed U3: SRV05-4, Package_TO_SOT_SMD:SOT-23-6_Handsoldering, symbol Power_Protection:SRV05-4
- removed U4: E22P-868M30S, E22-900M30S:XCVR_E22-900M30S, symbol New_Library:E22P-868M30S
- removed U5: ESP32-S3-WROOM-1, Library:ESP32-S3-WROOM-1, symbol RF_Module:ESP32-S3-WROOM-1
- added AE1: Antenna_Shield, Connector_Coaxial:SMA_Amphenol_132289_EdgeMount, symbol Device:Antenna_Shield
- added D2, D3: LED, LED_SMD:LED_0603_1608Metric_Pad1.05x0.95mm_HandSolder, symbol Device:LED
- added J1: USB_C_Receptacle_USB2.0_16P, Connector_USB:USB_C_Receptacle_GCT_USB4105-xx-A_16P_TopMnt_Horizontal, symbol Connector:USB_C_Receptacle_USB2.0_16P
- added R3, R6, R7: 1k, Resistor_SMD:R_0603_1608Metric_Pad0.98x0.95mm_HandSolder, symbol Device:R
- added R4, R5, R8, R9: 5.1k, Resistor_SMD:R_0603_1608Metric_Pad0.98x0.95mm_HandSolder, symbol Device:R
- added SW2: SW_SPDT, Button_Switch_SMD:SW_SPDT_PCM12, symbol Switch:SW_SPDT
- added U2: AP2112K-3.3, Package_TO_SOT_SMD:SOT-23-5, symbol Regulator_Linear:AP2112K-3.3
- added U3: E22-900MM22S, Library:E22-900MM22S, symbol New_Library:E22-900MM22S
- added U4: MCP73831-2-OT, Package_TO_SOT_SMD:SOT-23-5, symbol Battery_Management:MCP73831-2-OT
- C3: value 10uF -> 100nF; footprint Capacitor_SMD:C_1206_3216Metric_Pad1.33x1.80mm_HandSolder -> Capacitor_SMD:C_0603_1608Metric_Pad1.08x0.95mm_HandSolder
- D1: footprint LED_THT:LED_D3.0mm -> LED_SMD:LED_0603_1608Metric_Pad1.05x0.95mm_HandSolder
- R1: footprint (none) -> Resistor_SMD:R_0603_1608Metric_Pad0.98x0.95mm_HandSolder
- R2: value 100k -> R; LCSC C25803 -> (none)
Connections:
- net EN is gone; now on net GND: R2.2
- net +3.3V: now also U2.5 (VOUT); no longer C2.1
- net +5V: now also J1.A4 (VBUS), J1.A9 (VBUS), J1.B4 (VBUS), J1.B9 (VBUS), U4.4 (V_{DD})
- net BUSY: now also U3.11 (BUSY)
- net CS: now also U3.14 (NSS)
- net GND: now also AE1.2 (Shield), D2.1 (K), D3.1 (K), J1.A1 (GND), J1.A12 (GND), J1.B1 (GND), J1.B12 (GND), J1.S1 (SHIELD), R4.2, R8.2, R9.2, U2.2 (GND), U3.16 (GND), U3.2 (GND), U3.7 (GND), U4.2 (V_{SS})
- net IRQ: now also U3.20 (DIO1)
- net MISO: now also U3.12 (MISO)
- net MOSI: now also U3.13 (MOSI)
- net RXEN: now also U3.10 (RXEN)
- net SCK: now also U3.15 (SCK)
- net TXEN: now also U3.19 (DIO2), U3.9 (TXEN)
- net at D1.2 (A): now also R6.2; no longer R1.2
- net BAT+: now reaches R1.1
- net +3V3 renamed BAT_SENSE
- net BAT_SENSE: now also R1.2; no longer C3.1
- new net: D2.2 (A), R3.2
- new net: R6.1, U4.1 (STAT)
- new net: R4.1, U4.5 (PROG)
- new net: J1.B5 (CC2), R8.1
- new net: D3.2 (A), R7.2
- new net: J1.A5 (CC1), R9.1
- new net +BATT: SW2.2 (B), U4.3 (V_{BAT})
- new net ANT: AE1.1 (A), U3.6 (ANT)
- new net D+: J1.A6 (D+), J1.B6 (D+)
- new net D-: J1.A7 (D-), J1.B7 (D-)
- new net E22_RST: U3.3 (NRST)
- new net E22_VCC: C2.1, C3.1, U3.1 (VCC)
- new net LED: R7.1
- new net REG_EN: R5.1, U2.3 (EN)
- new net VCC: R3.1, R5.2, SW2.1 (A), U2.1 (VIN)
- no-connect marks 13 -> 8
Other:
- note removed: "1.8V"

Commit message: small ordered v1
Parts:
- removed H1, H2: MountingHole, MountingHole:MountingHole_2.2mm_M2_Pad_Via, symbol Mechanical:MountingHole
- removed J3: UART, Connector_PinHeader_2.54mm:PinHeader_1x04_P2.54mm_Vertical, symbol Connector_Generic:Conn_01x04
- added C1, C4, C5, C6: 10uF, Capacitor_SMD:C_0603_1608Metric_Pad1.08x0.95mm_HandSolder, symbol Device:C
- added J2: Conn_01x02_Shielded, Connector_JST:JST_SH_SM02B-SRSS-TB_1x02-1MP_P1.00mm_Horizontal, symbol Connector_Generic_Shielded:Conn_01x02_Shielded
- added J3: Conn_01x05, Connector_PinHeader_2.54mm:PinHeader_1x05_P2.54mm_Vertical, symbol Connector_Generic:Conn_01x05
- added J4: Conn_01x02, Library:1x02 smd 2.54, symbol Connector_Generic:Conn_01x02
- added L1: 10uH, Inductor_SMD:L_0603_1608Metric_Pad1.05x0.95mm_HandSolder, symbol Device:L
- added R10: 5.1k, Resistor_SMD:R_0603_1608Metric_Pad0.98x0.95mm_HandSolder, symbol Device:R
- added SW1: SW_Push, Button_Switch_SMD:SW_SPST_B3U-1000P, symbol Switch:SW_Push
- added U1: E73-2G4M08S1C, Library:E22-900MM22S_handsolder, symbol E73-2G4M08S1C:E73-2G4M08S1C
- C2: value 10uF -> 100nF; footprint Capacitor_SMD:C_1206_3216Metric_Pad1.33x1.80mm_HandSolder -> Capacitor_SMD:C_0603_1608Metric_Pad1.08x0.95mm_HandSolder
- R1, R2: value R -> 1M
- U2, U4: footprint Package_TO_SOT_SMD:SOT-23-5 -> Package_TO_SOT_SMD:SOT-23-5_HandSoldering
Connections:
- net BAT+ is gone; now on net VCC: R1.1
- net +3.3V: now also C3.1, U3.1 (VCC), C1.1
- net +5V: now also C6.1, J4.2 (Pin_2), U1.27 (VBUS)
- net +BATT: now also C5.1, J2.2 (Pin_2)
- net BAT_SENSE: now also C2.1, U1.4 (P0.28/AIN4)
- net BUSY: now also U1.6 (P1.13)
- net CS: now also U1.9 (P0.31/AIN7)
- net D+: now also U1.31 (DP)
- net D-: now also U1.29 (DM)
- net E22_RST: now also U1.1 (P1.11)
- net GND: now also C1.2, C4.2, C5.2, C6.2, J2.1 (Pin_1), J3.1 (Pin_1), J4.1 (Pin_1), SW1.1, U1.21 (GND@2), U1.24 (GND@3), U1.5 (GND@1)
- net IRQ: now also U1.3 (P0.03/AIN1)
- net LED: now also U1.15 (P0.05/AIN3)
- net MISO: now also U1.7 (P0.02/AIN0)
- net MOSI: now also U1.8 (P0.29/AIN5)
- net RXEN: now also U1.17 (P1.09)
- net SCK: now also U1.10 (P0.30/AIN6)
- net VCC: now also C4.1, U1.23 (VDDH)
- removed net E22_VCC: C2.1, C3.1, U3.1 (VCC)
- new net: L1.1, U1.25 (DCCH)
- new net NRF_RESET: J3.4 (Pin_4), R10.2, SW1.2, U1.26 (P0.18/RESET)
- new net SWDCLK: J3.2 (Pin_2), U1.39 (SWDCLK)
- new net SWDIO: J3.3 (Pin_3), U1.37 (SWDIO)
- new net VDD: J3.5 (Pin_5), L1.2, R10.1, U1.19 (VDD)
- no-connect marks 8 -> 10
Other:
- moved on the sheet: AE1, C3, D1, J1, R1, R2, R4, R5, R6, R8, R9, SW2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

Commit message: v2 rc1
Parts:
- removed D3: LED, LED_SMD:LED_0603_1608Metric_Pad1.05x0.95mm_HandSolder, symbol Device:LED
- removed R7: 1k, Resistor_SMD:R_0603_1608Metric_Pad0.98x0.95mm_HandSolder, symbol Device:R
- added BZ1: Buzzer, Library:MLT-5020, symbol Device:Buzzer
- added C7: 10uF, Capacitor_SMD:C_0603_1608Metric_Pad1.08x0.95mm_HandSolder, symbol Device:C
- added Q1: AO3400A, Package_TO_SOT_SMD:SOT-23_Handsoldering, symbol Transistor_FET:AO3400A
- C1: renamed from C3; footprint Capacitor_SMD:C_0603_1608Metric_Pad1.08x0.95mm_HandSolder -> Capacitor_SMD:C_0402_1005Metric_Pad0.74x0.62mm_HandSolder
- C2: footprint Capacitor_SMD:C_0603_1608Metric_Pad1.08x0.95mm_HandSolder -> Capacitor_SMD:C_0402_1005Metric_Pad0.74x0.62mm_HandSolder
- R5: value 5.1k -> 10k
- R6: renamed from R10; value 5.1k -> 10k
- U1: footprint Library:E22-900MM22S_handsolder -> Library:E73-2G4M08S1C
- U3: footprint Library:E22-900MM22S -> Library:E22-900MM22S_handsolder
- renumbered C1 to C3, R6 to R4, R4 to R7
Connections:
- net +3.3V: now also BZ1.1 (+), C7.1
- net +5V: now also D1.2 (A)
- net GND: now also J2.MP (Shield), C7.2, Q1.2 (S); no longer D1.1 (K)
- net LED: now also R3.1
- net REG_EN: now also U1.33 (P0.13)
- net VCC: no longer R3.1
- net at R4.1: now also D1.1 (K); no longer U4.1 (STAT)
- net STAT: now reaches R4.2
- net STAT: now also U4.1 (STAT); no longer D1.2 (A)
- net BUZZER: now reaches U1.2 (P1.10)
- net BUZZER: now also Q1.1 (G)
- new net: BZ1.2 (-), Q1.3 (D)
- no-connect marks 10 -> 5
Other:
- moved on the sheet: C2, C3, C4, C5, C6, D1, D2, J1, J2, J4, R1, R2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

Commit message: v2 rc2
Parts:
- J4: value Conn_01x02 -> Qi Charger; footprint Library:1x02 smd 2.54 -> Library:QiCharger
- R3: renamed from R5; value 10k -> 1M
- R4: value 1k -> 330
- R5: renamed from R3; value 1k -> 330
- R6: value 10k -> 5.1k
- U3: footprint Library:E22-900MM22S_handsolder -> Library:E22-900MM22S
Connections:
- net GND: now also R3.1, U3.17 (NC), U3.4 (NC), U3.5 (NC), U3.8 (NC)
- net REG_EN: now also R3.2; no longer R3.1
- net VCC: no longer R3.2
- no-connect marks 5 -> 6
Other:
- moved on the sheet: R3
Changed lines of the file:
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@@
 	)
 	(junction
-		(at 233.68 113.03)
+		(at 54.61 157.48)
 		(diameter 0)
 		(color 0 0 0 0)
 	)
 	(junction
-		(at 54.61 157.48)
+		(at 237.49 128.27)
 		(diameter 0)
 		(color 0 0 0 0)
@@
 	)
 	(junction
-		(at 233.68 120.65)
+		(at 262.89 118.11)
 		(diameter 0)
 		(color 0 0 0 0)
 	)
 	(junction
-		(at 262.89 118.11)
+		(at 39.37 167.64)
 		(diameter 0)
 		(color 0 0 0 0)
 	)
 	(junction
-		(at 39.37 167.64)
+		(at 185.42 91.44)
 		(diameter 0)
 		(color 0 0 0 0)
 	)
 	(junction
-		(at 185.42 91.44)
+		(at 74.93 53.34)
+		(diameter 0)
+		(color 0 0 0 0)
+	)
+	(junction
+		(at 52.07 55.88)
 		(diameter 0)
 		(color 0 0 0 0)
@@
 		(color 0 0 0 0)
 	)
+	(junction
+		(at 52.07 49.53)
+		(diameter 0)
+		(color 0 0 0 0)
+	)
+	(junction
+		(at 237.49 120.65)
+		(diameter 0)
+		(color 0 0 0 0)
+	)
 	(no_connect
 		(at 227.33 90.17)
@@
 	)
 	(no_connect
+		(at 110.49 127)
+	)
+	(no_connect
 		(at 110.49 129.54)
 	)
@@
 	(wire
 		(pts
+			(xy 237.49 128.27) (xy 222.25 128.27)
+		)
+		(stroke
+			(width 0)
+			(type default)
+		)
+	)
+	(wire
+		(pts
 			(xy 54.61 157.48) (xy 54.61 160.02)
 		)
@@
 	(wire
 		(pts
-			(xy 229.87 113.03) (xy 233.68 113.03)
+			(xy 229.87 113.03) (xy 241.3 113.03)
 		)
 		(stroke
@@
 	(wire
 		(pts
-			(xy 233.68 120.65) (xy 242.57 120.65)
+			(xy 52.07 49.53) (xy 52.07 50.8)
 		)
 		(stroke
@@
 	(wire
 		(pts
+			(xy 41.91 49.53) (xy 52.07 49.53)
+		)
+		(stroke
+			(width 0)
+			(type default)
+		)
+	)
+	(wire
+		(pts
 			(xy 191.77 33.02) (xy 191.77 34.29)
 		)
@@
 	(wire
 		(pts
+			(xy 74.93 53.34) (xy 74.93 55.88)
+		)
+		(stroke
+			(width 0)
+			(type default)
+		)
+	)
+	(wire
+		(pts
 			(xy 190.5 35.56) (xy 191.77 35.56)
 		)
@@
 	(wire
 		(pts
+			(xy 52.07 48.26) (xy 52.07 49.53)
+		)
+		(stroke
+			(width 0)
+			(type default)
+		)
+	)
+	(wire
+		(pts
 			(xy 222.25 120.65) (xy 222.25 113.03)
 		)
@@
 	(wire
 		(pts
-			(xy 231.14 120.65) (xy 233.68 120.65)
+			(xy 231.14 120.65) (xy 237.49 120.65)
 		)
 		(stroke
@@
 	(wire
 		(pts
-			(xy 250.19 128.27) (xy 222.25 128.27)
+			(xy 52.07 55.88) (xy 52.07 58.42)
 		)
 		(stroke
@@
 	(wire
 		(pts
-			(xy 191.77 34.29) (xy 191.77 35.56)
+			(xy 250.19 128.27) (xy 237.49 128.27)
 		)
 		(stroke
@@
 	(wire
 		(pts
-			(xy 173.99 45.72) (xy 173.99 46.99)
+			(xy 191.77 34.29) (xy 191.77 35.56)
 		)
 		(stroke
@@
 	(wire
 		(pts
-			(xy 233.68 113.03) (xy 241.3 113.03)
+			(xy 173.99 45.72) (xy 173.99 46.99)
 		)
 		(stroke
@@
 	(wire
 		(pts
+			(xy 237.49 120.65) (xy 242.57 120.65)
+		)
+		(stroke
+			(width 0)
+			(type default)
+		)
+	)
+	(wire
+		(pts
 			(xy 173.99 46.99) (xy 173.99 48.26)
 		)
@@
 		(dnp no)
 		(fields_autoplaced yes)
-		(property "Reference" "R3"
+		(property "Reference" "R5"
 			(at 149.86 92.7099 0)
 			(show_name no)
@@
 			)
 		)
-		(property "Value" "1k"
+		(property "Value" "330"
 			(at 149.86 95.2499 0)
 			(show_name no)
@@
 			(project "lora_board"
 				(path "/29f0db4c-6d53-4dfd-90c6-c907c21b419f"
-					(reference "R3")
+					(reference "R5")
 					(unit 1)
 				)
@@
 			)
 		)
-		(property "Value" "1k"
+		(property "Value" "330"
 			(at 259.08 66.0399 0)
 			(show_name no)
@@
 	)
 	(symbol
+		(lib_id "power:GND")
+		(at 41.91 49.53 0)
+		(unit 1)
+		(body_style 1)
+		(exclude_from_sim no)
+		(in_bom yes)
+		(on_board yes)
+		(in_pos_files yes)
+		(dnp no)
+		(fields_autoplaced yes)
+		(property "Reference" "#PWR040"
+			(at 41.91 55.88 0)
+			(hide yes)
+			(show_name no)
+			(do_not_autoplace no)
+			(effects
+				(font
+					(size 1.27 1.27)
+				)
+			)
+		)
+		(property "Value" "GND"
+			(at 41.91 54.61 0)
+			(show_name no)
+			(do_not_autoplace no)
+			(effects
+				(font
+					(size 1.27 1.27)
+				)
+			)
+		)
+		(property "Footprint" ""
+			(at 41.91 49.53 0)
+			(hide yes)
+			(show_name no)
+			(do_not_autoplace no)
+			(effects
+				(font
+					(size 1.27 1.27)
+				)
+			)
+		)
+		(property "Datasheet" ""
+			(at 41.91 49.53 0)
+			(hide yes)
+			(show_name no)
+			(do_not_autoplace no)
+			(effects
+				(font
+					(size 1.27 1.27)
+				)
+			)
+		)
+		(property "Description" "Power symbol creates a global label with name \"GND\" , ground"
+			(at 41.91 49.53 0)
+			(hide yes)
+			(show_name no)
+			(do_not_autoplace no)
+			(effects
+				(font
+					(size 1.27 1.27)
+				)
+			)
+		)
+		(pin "1"
+		)
+		(instances
+			(project "lora_board"
+				(path "/29f0db4c-6d53-4dfd-90c6-c907c21b419f"
+					(reference "#PWR040")
+					(unit 1)
+				)
+			)
+		)
+	)
+	(symbol
 		(lib_id "Regulator_Linear:AP2112K-3.3")
 		(at 250.19 120.65 0)
@@
 			)
 		)
-		(property "Value" "10k"
+		(property "Value" "5.1k"
 			(at 41.91 162.5599 0)
 			(show_name no)
@@
 	(symbol
 		(lib_id "Device:R")
-		(at 233.68 116.84 180)
+		(at 237.49 124.46 180)
 		(unit 1)
 		(body_style 1)
@@
 		(dnp no)
 		(fields_autoplaced yes)
-		(property "Reference" "R5"
-			(at 236.22 115.5699 0)
+		(property "Reference" "R3"
+			(at 240.03 123.1899 0)
 			(show_name no)
 			(do_not_autoplace no)
@@
 			)
 		)
-		(property "Value" "10k"
-			(at 236.22 118.1099 0)
+		(property "Value" "1M"
+			(at 240.03 125.7299 0)
 			(show_name no)
 			(do_not_autoplace no)
@@
 		)
 		(property "Footprint" "Resistor_SMD:R_0603_1608Metric_Pad0.98x0.95mm_HandSolder"
-			(at 235.458 116.84 90)
+			(at 239.268 124.46 90)
 			(hide yes)
 			(show_name no)
@@
 		)
 		(property "Datasheet" ""
-			(at 233.68 116.84 0)
+			(at 237.49 124.46 0)
 			(hide yes)
 			(show_name no)
@@
 		)
 		(property "Description" "Resistor"
-			(at 233.68 116.84 0)
+			(at 237.49 124.46 0)
 			(hide yes)
 			(show_name no)
@@
 		)
 		(property "MANUFACTURER" ""
-			(at 233.68 116.84 0)
+			(at 237.49 124.46 0)
 			(hide yes)
 			(show_name no)
@@
 		)
 		(property "MAXIMUM_PACKAGE_HEIGHT" ""
-			(at 233.68 116.84 0)
+			(at 237.49 124.46 0)
 			(hide yes)
 			(show_name no)
@@
 		)
 		(property "PARTREV" ""
-			(at 233.68 116.84 0)
+			(at 237.49 124.46 0)
 			(hide yes)
 			(show_name no)
@@
 		)
 		(property "STANDARD" ""
-			(at 233.68 116.84 0)
+			(at 237.49 124.46 0)
 			(hide yes)
 			(show_name no)
@@
 			(project "lora_board"
 				(path "/29f0db4c-6d53-4dfd-90c6-c907c21b419f"
-					(reference "R5")
+					(reference "R3")
 					(unit 1)
 				)
@@
 			)
 		)
-		(property "Footprint" "Library:E22-900MM22S_handsolder"
+		(property "Footprint" "Library:E22-900MM22S"
 			(at 63.5 52.07 0)
 			(hide yes)
@@
 			)
 		)
-		(property "Value" "Conn_01x02"
+		(property "Value" "Qi Charger"
 			(at 58.42 113.03 0)
 			(show_name no)
@@
 			)
 		)
-		(property "Footprint" "Library:1x02 smd 2.54"
+		(property "Footprint" "Library:QiCharger"
 			(at 58.42 119.38 0)
 			(hide yes)
