File: pcb/lora_board.kicad_pcb (KiCad board)
At the start: 2 copper layers, 20 x 45 mm, 32 parts, among them J1 USB_C_Receptacle_USB2.0_16P, J2 Conn_01x02_Shielded, J3 Conn_01x05, J4 Qi Charger, Q1 AO3400A, SW1 SW_Push, SW2 SW_SPDT, U1 E73-2G4M08S1C, U2 AP2112K-3.3, U3 E22-900MM22S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

Commit message: v2 rc3
Parts:
- Q1: footprint Package_TO_SOT_SMD:SOT-23_Handsoldering -> Package_TO_SOT_SMD:SOT-23-3
- U2, U4: footprint Package_TO_SOT_SMD:SOT-23-5_HandSoldering -> Package_TO_SOT_SMD:SOT-23-5
- moved C2 1.03 mm to (107.8, 94.2), turned to 90 degrees
- moved U2 0.90 mm to (103.5, 93.0)
- moved BZ1 0.50 mm to (99.0, 87.0)
- moved C7 0.50 mm to (96.5, 91.2)
- moved C1 0.35 mm to (110.8, 93.8)
- moved R3 0.25 mm to (97.0, 95.5)
- moved SW2 0.25 mm to (100.2, 77.0)
- moved Q1 0.10 mm to (99.3, 91.2)
Routing:
- net VCC: track 42.1 -> 43.6 mm
- net /REG_EN: track 23.3 -> 24.1 mm
- net /BAT_SENSE: track 22.9 -> 22.2 mm
- net GND: vias 46 -> 49

Commit message: ordered v2
Parts:
- moved AE1 15.0 mm to (126.0, 77.5)
- moved BZ1 15.0 mm to (114.0, 87.0)
- moved C1 15.0 mm to (125.8, 93.8)
- moved C2 15.0 mm to (122.8, 94.2)
- moved C3 15.0 mm to (124.2, 94.0)
- moved C4 15.0 mm to (112.0, 94.0)
- moved C5 15.0 mm to (128.0, 111.8)
- moved C6 15.0 mm to (124.5, 111.5)
- moved C7 15.0 mm to (111.5, 91.2)
- moved D1 15.0 mm to (128.0, 119.0)
- moved D2 15.0 mm to (112.0, 119.0)
- moved J1 15.0 mm to (119.2, 117.5)
- moved J2 15.0 mm to (116.0, 82.0)
- moved J3 15.0 mm to (125.6, 103.0)
- moved J4 15.0 mm to (120.5, 80.0)
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Routing:
- net (no net): track 0.00 -> 10.5 mm
- net GND: vias 49 -> 51
- net /TXEN: vias 0 -> 2
Other:
- board text added: "LORA BATTERY NODE v2"
- board text removed: "LSBN v2"
