File: pcb/lora_board.kicad_sch (KiCad schematic)
At the start: 32 parts, among them J1 USB_C_Receptacle_USB2.0_16P, J2 Conn_01x02_Shielded, J3 Conn_01x05, J4 Qi Charger, Q1 AO3400A, SW1 SW_Push, SW2 SW_SPDT, U1 E73-2G4M08S1C, U2 AP2112K-3.3, U3 E22-900MM22S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

Commit message: v2 rc3
Connections:
- no-connect marks 6 -> 20
Changed lines of the file:
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@@
+	)
+	(no_connect
+		(at 110.49 144.78)
 	)
 	(no_connect
@@
 	)
 	(no_connect
+		(at 110.49 142.24)
+	)
+	(no_connect
+		(at 137.16 152.4)
+	)
+	(no_connect
+		(at 110.49 137.16)
+	)
+	(no_connect
+		(at 137.16 144.78)
+	)
+	(no_connect
+		(at 110.49 160.02)
+	)
+	(no_connect
+		(at 110.49 154.94)
+	)
+	(no_connect
 		(at 110.49 129.54)
 	)
 	(no_connect
+		(at 110.49 162.56)
+	)
+	(no_connect
+		(at 110.49 165.1)
+	)
+	(no_connect
+		(at 110.49 172.72)
+	)
+	(no_connect
+		(at 110.49 167.64)
+	)
+	(no_connect
+		(at 110.49 147.32)
+	)
+	(no_connect
+		(at 137.16 147.32)
+	)
+	(no_connect
+		(at 137.16 149.86)
+	)
+	(no_connect

Commit message: ordered v2
Other:
- moved on the sheet: AE1, BZ1, C1, C2, C3, C4, C5, C6, C7, D1, D2, J1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
